File: pcb-main/oa_sevenfortyfun.brd (EAGLE design)
At the start: 88.9 x 71.1 mm, 46 parts, among them J1 1X01-TERM, J2 1X01-TERM, J3 1X01-TERM, J4 1X01-TERM, J5 1X01-TERM, J6 1X01-TERM, J7 1X01-TERM, J8 1X01-TERM, J9 2X04SHR, Q1 2N3904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

Commit message: updated files
Parts:
- STANDOFF1, STANDOFF2, STANDOFF3, STANDOFF4: value STAND-OFF -> STAND-OFF4; device Ai_Electromechanical:STAND-OFF -> Ai_Electromechanical:STAND-OFF-4
Routing:
- net VCC-: track 82.6 -> 0.00 mm, vias 1 -> 0
- net N$15: track 31.8 -> 31.2 mm
Other:
- board text added: "v1.2"
- board text removed: "v1.1"
